File: pcb/controll.kicad_sc.kicad_sch (KiCad schematic)
At the start: 5 parts, among them SW4 SW_Push

Commit message: Add files via upload
Connections:
- net GND: no longer SW4.2
- net ADC: now reaches RN2.2
- new net SW4: SW4.2
- no-connect marks 2 -> 0
Other:
- moved on the sheet: SW4
Changed lines of the file:
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@@
 	(paper "A4")
-	(junction
-		(at 151.13 93.98)
-		(diameter 0)
-		(color 0 0 0 0)
-	)
 	(junction
 		(at 124.46 93.98)
@@
 		(color 0 0 0 0)
 	)
-	(no_connect
-		(at 116.84 105.41)
-	)
-	(no_connect
-		(at 152.4 93.98)
-	)
 	(wire
 		(pts
-			(xy 151.13 93.98) (xy 152.4 93.98)
+			(xy 123.19 101.6) (xy 124.46 101.6)
 		)
 		(stroke
@@
 	(wire
 		(pts
-			(xy 123.19 101.6) (xy 124.46 101.6)
+			(xy 124.46 93.98) (xy 127 93.98)
 		)
 		(stroke
@@
 	(wire
 		(pts
-			(xy 124.46 93.98) (xy 151.13 93.98)
+			(xy 113.03 93.98) (xy 116.84 93.98)
 		)
 		(stroke
@@
 		)
 	)
-	(wire
-		(pts
-			(xy 113.03 93.98) (xy 116.84 93.98)
-		)
-		(stroke
-			(width 0)
-			(type default)
+	(hierarchical_label "SW4"
+		(shape input)
+		(at 137.16 93.98 0)
+		(effects
+			(font
+				(size 1.27 1.27)
+			)
+			(justify left)
+		)
+	)
+	(hierarchical_label "ADC"
+		(shape input)
+		(at 116.84 105.41 270)
+		(effects
+			(font
+				(size 1.27 1.27)
+			)
+			(justify right)
 		)
 	)
@@
 	(symbol
 		(lib_id "Switch:SW_Push")
-		(at 151.13 88.9 90)
+		(at 132.08 93.98 0)
 		(unit 1)
 		(body_style 1)
@@
 		(in_pos_files yes)
 		(dnp no)
-		(fields_autoplaced yes)
 		(property "Reference" "SW4"
-			(at 152.4 87.6299 90)
+			(at 133.3501 95.25 90)
 			(show_name no)
 			(do_not_autoplace no)
@@
 		)
 		(property "Value" "SW_Push"
-			(at 152.4 90.1699 90)
+			(at 135.636 89.154 0)
 			(show_name no)
 			(do_not_autoplace no)
@@
 		)
 		(property "Footprint" "Button_Switch_SMD:SW_Push_1TS009xxxx-xxxx-xxxx_6x6x5mm"
-			(at 146.05 88.9 0)
+			(at 132.08 88.9 0)
 			(hide yes)
 			(show_name no)
@@
 		)
 		(property "Datasheet" ""
-			(at 146.05 88.9 0)
+			(at 132.08 88.9 0)
 			(hide yes)
 			(show_name no)
@@
 		)
 		(property "Description" "Push button switch, generic, two pins"
-			(at 151.13 88.9 0)
+			(at 132.08 93.98 0)
 			(hide yes)
 			(show_name no)
@@
 					(unit 1)
 				)
-			)
-		)
-	)
-	(symbol
-		(lib_id "power:GND")
-		(at 151.13 83.82 90)
-		(unit 1)
-		(body_style 1)
-		(exclude_from_sim no)
-		(in_bom yes)
-		(on_board yes)
-		(in_pos_files yes)
-		(dnp no)
-		(fields_autoplaced yes)
-		(property "Reference" "#PWR023"
-			(at 157.48 83.82 0)
-			(hide yes)
-			(show_name no)
-			(do_not_autoplace no)
-			(effects
-				(font
-					(size 1.27 1.27)
-				)
-			)
-		)
-		(property "Value" "GND"
-			(at 154.94 83.8199 90)
-			(show_name no)
-			(do_not_autoplace no)
-			(effects
-				(font
-					(size 1.27 1.27)
-				)
-				(justify right)
-			)
-		)
-		(property "Footprint" ""
-			(at 151.13 83.82 0)
-			(hide yes)
-			(show_name no)
-			(do_not_autoplace no)
-			(effects
-				(font
-					(size 1.27 1.27)
-				)
-			)
-		)
-		(property "Datasheet" ""
-			(at 151.13 83.82 0)
-			(hide yes)
-			(show_name no)
-			(do_not_autoplace no)
-			(effects
-				(font
-					(size 1.27 1.27)
-				)
-			)
-		)
-		(property "Description" "Power symbol creates a global label with name \"GND\" , ground"
-			(at 151.13 83.82 0)
-			(hide yes)
-			(show_name no)
-			(do_not_autoplace no)
-			(effects
-				(font
-					(size 1.27 1.27)
-				)
-			)
-		)
-		(pin "1"
-		)
-		(instances
-			(project "kiki-player"
-				(path "/a20a05c5-243f-410a-9881-de77a274e6b8/572b974a-9196-4f58-b937-aee5588a958e"
-					(reference "#PWR023")
-					(unit 1)
-				)
