File: pcb/kiki-player.kicad_sch (KiCad schematic)
At the start: 24 parts, among them J2 Conn_01x28_Socket, J3 AudioPlug3, J4 SD_Card_Device, J5 Conn_02x01, J6 USB_C_Receptacle_USB2.0_16P, U1 ESP32-S3-WROOM-1, U4 CR2013-MI2120, U5 PCM5102A, U6 MAX98357A, U7 DS3231M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

Commit message: Add files via upload
Parts:
- added C1, C4: 100nf, symbol Device:C
- added C2, C3: 10uF, symbol Device:C
- J2: value Conn_01x28_Socket -> MGC3031
Connections:
- net +3V3: now also C1.2, C2.2, C3.2, C4.2
- net GND: now also C8.2, C1.1, C2.1, C3.1, C4.1; no longer C8.1
- net Tip: now also C14.1; no longer C14.2
- net VBAT: now also U7.14 (VBAT)
- net at Y1.1: now also C8.1; no longer C8.2
- net at J3.T: now also C14.2; no longer C14.1
- net ADC: now reaches U1.12 (IO8)
- net SW3: now reaches U1.8 (IO15)
- net SW4: now reaches U1.9 (IO16)
- net CLK renamed SCK
- net DAT0 renamed MISO
- net DAT3: no longer names the net of J4.1 (CD/DAT3)
- net INT: no longer names the net of U7.3 (~{INT}/SQW)
- no-connect marks 57 -> 52
Other:
- sheet button ports: added SW3; removed none
- sheet controll ports: added ADC, SW4; removed none
- moved on the sheet: C12, C13, C14, C15, C16, C17, C18, C19, C7, C8, J2, J3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
