File: pcb/untitled.kicad_sch (KiCad schematic)
At the start: 3 parts, among them SW3 SW_Push

Commit message: Add files via upload
Connections:
- net GND: no longer C9.1, R6.1, R6.2, SW3.1, SW3.2
- new net: C9.1, SW3.2
- new net +3V3: R6.2
- new net SW3: R6.1, SW3.1
- no-connect marks 1 -> 0
Other:
- moved on the sheet: C9, SW3
